File: Inline SCART Splitter.kicad_pcb (KiCad board)
At the start: 2 copper layers, 59 x 49.8 mm, 40 parts, among them J1 SCART-F, J2 USB_B_Micro, J3 SCART-F, J4 SCART-F, U1 THS7374

Commit message: Finished board, added renders
Parts:
- added REF**: MountingHole_3.2mm_M3, MountingHole:MountingHole_3.2mm_M3, F.Cu at (106.0, 63.1)
- added REF**: MountingHole_3.2mm_M3, MountingHole:MountingHole_3.2mm_M3, F.Cu at (158.9, 63.1)
- moved J2 53.6 mm to (159.3, 41.3), turned to 90 degrees
- moved C1 17.2 mm to (113.3, 28.4)
- moved C2 17.2 mm to (113.3, 26.9)
- moved C4 17.2 mm to (151.1, 26.0)
- moved C5 17.2 mm to (141.8, 26.0)
- moved C6 17.2 mm to (134.1, 26.0)
- moved C7 17.2 mm to (126.5, 25.9)
- moved R1 17.2 mm to (151.1, 27.5)
- moved R2 17.2 mm to (141.8, 27.5)
- moved R3 17.2 mm to (134.1, 27.5)
- moved R4 17.2 mm to (126.5, 27.4)
- moved R5 17.2 mm to (151.1, 29.0)
- moved R6 17.2 mm to (141.8, 29.0)
- moved R7 17.2 mm to (134.1, 29.0)
- moved R8 17.2 mm to (126.5, 28.9)
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Routing:
- net Net-(FB1-Pad2): track 25.5 -> 54.6 mm
- net Net-(R13-Pad2): track 53.9 -> 74.7 mm, vias 2 -> 0
- net RED_IN: track 5.49 -> 23.6 mm
- net BLUE_IN: track 5.40 -> 22.8 mm
- net GREEN_IN: track 5.49 -> 22.5 mm
- net Net-(R12-Pad2): track 23.9 -> 40.3 mm
- net Net-(R11-Pad2): track 25.9 -> 42.3 mm, vias 2 -> 0
- net 5V: track 72.9 -> 88.4 mm, vias 1 -> 6
- net LEFT: track 45.5 -> 35.8 mm
- net Net-(R10-Pad2): track 37.6 -> 45.3 mm, vias 2 -> 0
- net RIGHT: track 39.3 -> 32.0 mm
- net SYNC_IN: track 10.6 -> 17.8 mm
- net Net-(C14-Pad2): track 10.8 -> 4.78 mm
- net Net-(C15-Pad2): track 13.7 -> 7.98 mm
- net Net-(C13-Pad2): track 12.4 -> 8.35 mm
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Other:
- board size 59 x 49.8 mm -> 59 x 42.7 mm

Commit message: generated gerbers
Routing:
- net GND: track 44.2 -> 54.0 mm
Changed lines of the file:
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@@
     (thickness 1.6)
     (drawings 5)
-    (tracks 320)
+    (tracks 327)
     (zones 0)
     (modules 42)
@@
     (pcbplotparams
       (layerselection 0x010fc_ffffffff)
-      (usegerberextensions false)
+      (usegerberextensions true)
       (usegerberattributes false)
       (usegerberadvancedattributes false)
@@
       (outputformat 1)
       (mirror false)
-      (drillshape 1)
+      (drillshape 0)
       (scaleselection 1)
-      (outputdirectory ""))
+      (outputdirectory "Gerbers/"))
   )
   (net 0 "")
@@
     (add_net SYNC_IN)
   )
-  (module MountingHole:MountingHole_3.2mm_M3 (layer F.Cu)
-    (at 106.05 63.15)
-    (descr "Mounting Hole 3.2mm, no annular, M3")
-    (tags "mounting hole 3.2mm no annular m3")
-    (attr virtual)
-    (fp_text reference REF** (at 0.15 -2.65) (layer F.SilkS) hide
-      (effects (font (size 1 1) (thickness 0.15)))
-    )
-    (fp_text value MountingHole_3.2mm_M3 (at 0 4.2) (layer F.Fab)
-      (effects (font (size 1 1) (thickness 0.15)))
-    )
-    (fp_circle (center 0 0) (end 1.765334 0) (layer F.CrtYd) (width 0.05))
-    (fp_circle (center 0 0) (end 1.765334 0) (layer Cmts.User) (width 0.15))
-    (fp_text user %R (at 0.3 0) (layer F.Fab)
-      (effects (font (size 1 1) (thickness 0.15)))
-    )
-    (pad "" np_thru_hole circle (at 0 0) (size 3.2 3.2) (drill 3.2) (layers *.Cu *.Mask))
-  )
-  (module MountingHole:MountingHole_3.2mm_M3 (layer F.Cu)
-    (at 158.95 63.15)
-    (descr "Mounting Hole 3.2mm, no annular, M3")
-    (tags "mounting hole 3.2mm no annular m3")
-    (attr virtual)
-    (fp_text reference REF** (at 0.15 -2.65) (layer F.SilkS) hide
-      (effects (font (size 1 1) (thickness 0.15)))
-    )
-    (fp_text value MountingHole_3.2mm_M3 (at 0 4.2) (layer F.Fab)
-      (effects (font (size 1 1) (thickness 0.15)))
-    )
-    (fp_text user %R (at 0.3 0) (layer F.Fab)
-      (effects (font (size 1 1) (thickness 0.15)))
-    )
-    (fp_circle (center 0 0) (end 1.765334 0) (layer Cmts.User) (width 0.15))
-    (fp_circle (center 0 0) (end 1.765334 0) (layer F.CrtYd) (width 0.05))
-    (pad "" np_thru_hole circle (at 0 0) (size 3.2 3.2) (drill 3.2) (layers *.Cu *.Mask))
-  )
-  (module MountingHole:MountingHole_3.2mm_M3 (layer F.Cu)
-    (at 106.05 26.55)
-    (descr "Mounting Hole 3.2mm, no annular, M3")
-    (tags "mounting hole 3.2mm no annular m3")
-    (attr virtual)
-    (fp_text reference REF** (at 0.15 -2.65) (layer F.SilkS) hide
-      (effects (font (size 1 1) (thickness 0.15)))
-    )
-    (fp_text value MountingHole_3.2mm_M3 (at 0 4.2) (layer F.Fab)
-      (effects (font (size 1 1) (thickness 0.15)))
-    )
-    (fp_text user %R (at 0.3 0) (layer F.Fab)
-      (effects (font (size 1 1) (thickness 0.15)))
-    )
-    (fp_circle (center 0 0) (end 1.765334 0) (layer Cmts.User) (width 0.15))
-    (fp_circle (center 0 0) (end 1.765334 0) (layer F.CrtYd) (width 0.05))
-    (pad "" np_thru_hole circle (at 0 0) (size 3.2 3.2) (drill 3.2) (layers *.Cu *.Mask))
-  )
-  (module MountingHole:MountingHole_3.2mm_M3 (layer F.Cu)
-    (at 158.95 26.55)
-    (descr "Mounting Hole 3.2mm, no annular, M3")
-    (tags "mounting hole 3.2mm no annular m3")
-    (attr virtual)
-    (fp_text reference REF** (at 0.15 -2.65) (layer F.SilkS) hide
-      (effects (font (size 1 1) (thickness 0.15)))
-    )
-    (fp_text value MountingHole_3.2mm_M3 (at 0 4.2) (layer F.Fab)
-      (effects (font (size 1 1) (thickness 0.15)))
-    )
-    (fp_circle (center 0 0) (end 1.765334 0) (layer F.CrtYd) (width 0.05))
-    (fp_circle (center 0 0) (end 1.765334 0) (layer Cmts.User) (width 0.15))
-    (fp_text user %R (at 0.3 0) (layer F.Fab)
-      (effects (font (size 1 1) (thickness 0.15)))
-    )
-    (pad "" np_thru_hole circle (at 0 0) (size 3.2 3.2) (drill 3.2) (layers *.Cu *.Mask))
-  )
   (module Connector_USB:USB_Micro-B_Molex-105017-0001 (layer F.Cu)
     (at 159.3 41.3 90)
@@
     (pad 6 smd rect (at -2.9 1.2375 90) (size 1.2 1.9) (layers F.Cu F.Mask)
       (net 2 GND))
+    (pad 6 thru_hole circle (at -2.5 -1.4625 90) (size 1.45 1.45) (drill 0.85) (layers *.Cu *.Mask)
+      (net 2 GND))
     (model ${KISYS3DMOD}/Connector_USB.3dshapes/USB_Micro-B_Molex-105017-0001.wrl
       (at (xyz 0 0 0))
@@
       (rotate (xyz 0 0 0))
     )
+  )
+  (module MountingHole:MountingHole_3.2mm_M3 (layer F.Cu)
+    (at 106.05 63.15)
+    (descr "Mounting Hole 3.2mm, no annular, M3")
+    (tags "mounting hole 3.2mm no annular m3")
+    (attr virtual)
+    (fp_text reference REF** (at 0.15 -2.65) (layer F.SilkS) hide
+      (effects (font (size 1 1) (thickness 0.15)))
+    )
+    (fp_text value MountingHole_3.2mm_M3 (at 0 4.2) (layer F.Fab)
+      (effects (font (size 1 1) (thickness 0.15)))
+    )
+    (fp_circle (center 0 0) (end 1.765334 0) (layer F.CrtYd) (width 0.05))
+    (fp_circle (center 0 0) (end 1.765334 0) (layer Cmts.User) (width 0.15))
+    (fp_text user %R (at 0.3 0) (layer F.Fab)
+      (effects (font (size 1 1) (thickness 0.15)))
+    )
+    (pad "" np_thru_hole circle (at 0 0) (size 3.2 3.2) (drill 3.2) (layers *.Cu *.Mask))
+  )
+  (module MountingHole:MountingHole_3.2mm_M3 (layer F.Cu)
+    (at 158.95 63.15)
+    (descr "Mounting Hole 3.2mm, no annular, M3")
+    (tags "mounting hole 3.2mm no annular m3")
+    (attr virtual)
+    (fp_text reference REF** (at 0.15 -2.65) (layer F.SilkS) hide
+      (effects (font (size 1 1) (thickness 0.15)))
+    )
+    (fp_text value MountingHole_3.2mm_M3 (at 0 4.2) (layer F.Fab)
+      (effects (font (size 1 1) (thickness 0.15)))
+    )
+    (fp_text user %R (at 0.3 0) (layer F.Fab)
+      (effects (font (size 1 1) (thickness 0.15)))
+    )
+    (fp_circle (center 0 0) (end 1.765334 0) (layer Cmts.User) (width 0.15))
+    (fp_circle (center 0 0) (end 1.765334 0) (layer F.CrtYd) (width 0.05))
+    (pad "" np_thru_hole circle (at 0 0) (size 3.2 3.2) (drill 3.2) (layers *.Cu *.Mask))
+  )
+  (module MountingHole:MountingHole_3.2mm_M3 (layer F.Cu)
+    (at 106.05 26.55)
+    (descr "Mounting Hole 3.2mm, no annular, M3")
+    (tags "mounting hole 3.2mm no annular m3")
+    (attr virtual)
+    (fp_text reference REF** (at 0.15 -2.65) (layer F.SilkS) hide
+      (effects (font (size 1 1) (thickness 0.15)))
+    )
+    (fp_text value MountingHole_3.2mm_M3 (at 0 4.2) (layer F.Fab)
+      (effects (font (size 1 1) (thickness 0.15)))
+    )
+    (fp_text user %R (at 0.3 0) (layer F.Fab)
+      (effects (font (size 1 1) (thickness 0.15)))
+    )
+    (fp_circle (center 0 0) (end 1.765334 0) (layer Cmts.User) (width 0.15))
+    (fp_circle (center 0 0) (end 1.765334 0) (layer F.CrtYd) (width 0.05))
+    (pad "" np_thru_hole circle (at 0 0) (size 3.2 3.2) (drill 3.2) (layers *.Cu *.Mask))
+  )
+  (module MountingHole:MountingHole_3.2mm_M3 (layer F.Cu)
+    (at 158.95 26.55)
+    (descr "Mounting Hole 3.2mm, no annular, M3")
+    (tags "mounting hole 3.2mm no annular m3")
+    (attr virtual)
+    (fp_text reference REF** (at 0.15 -2.65) (layer F.SilkS) hide
+      (effects (font (size 1 1) (thickness 0.15)))
+    )
+    (fp_text value MountingHole_3.2mm_M3 (at 0 4.2) (layer F.Fab)
+      (effects (font (size 1 1) (thickness 0.15)))
+    )
+    (fp_circle (center 0 0) (end 1.765334 0) (layer F.CrtYd) (width 0.05))
+    (fp_circle (center 0 0) (end 1.765334 0) (layer Cmts.User) (width 0.15))
+    (fp_text user %R (at 0.3 0) (layer F.Fab)
+      (effects (font (size 1 1) (thickness 0.15)))
+    )
+    (pad "" np_thru_hole circle (at 0 0) (size 3.2 3.2) (drill 3.2) (layers *.Cu *.Mask))
   )
   (module Capacitor_Tantalum_SMD:CP_EIA-7343-30_AVX-N_Pad2.25x2.55mm_HandSolder (layer B.Cu)
@@
   (via (at 116 31.4) (size 0.8) (drill 0.4) (layers F.Cu B.Cu) (net 2))
   (via (at 119.1 40.3) (size 0.8) (drill 0.4) (layers F.Cu B.Cu) (net 2))
+  (segment (start 157.8375 38.8) (end 157.8375 40) (width 0.25) (layer F.Cu) (net 2))
+  (segment (start 160.2375 40) (end 160.5375 40.3) (width 0.25) (layer F.Cu) (net 2))
+  (segment (start 157.8375 40) (end 160.2375 40) (width 0.25) (layer F.Cu) (net 2))
+  (segment (start 158.2375 38.4) (end 157.8375 38.8) (width 0.25) (layer F.Cu) (net 2))
+  (segment (start 160.5375 38.4) (end 158.2375 38.4) (width 0.25) (layer F.Cu) (net 2))
+  (segment (start 158.2375 44.2) (end 157.8375 43.8) (width 0.25) (layer F.Cu) (net 2))
+  (segment (start 160.5375 44.2) (end 158.2375 44.2) (width 0.25) (layer F.Cu) (net 2))
   (segment (start 149.750928 28.500928) (end 150.25 29) (width 0.25) (layer B.Cu) (net 3))
   (segment (start 149.1 27.85) (end 149.750928 28.500928) (width 0.25) (layer B.Cu) (net 3))
